Commit message: Refactor setup.py and my_robot.urdf for clarity and consistency

File: ros2_ws/src/my_robot_description/urdf/my_robot.urdf (robot description, URDF)
Before this commit: robot my_robot, 5 links, 4 joints
Joints:
- joint left_wheel_joint: axis 0 1 0 -> 0 0 1; origin xyz=-0.1 0.25 0 rpy=0 0 0 -> xyz=-0.1 0.25 0 rpy=-1.5708 0 0
- joint right_wheel_joint: axis 0 1 0 -> 0 0 1; origin xyz=-0.1 -0.25 0 rpy=0 0 0 -> xyz=-0.1 -0.25 0 rpy=-1.5708 0 0
