Commit message: Enhance my_robot.xacro with materials, geometry, and drive wheel macro for improved robot definition

File: ros2_ws/src/assignment2/urdf/my_robot .urdf.xacro (robot description, xacro)
@@ -1,3 +1,4 @@
 <?xml version="1.0"?>
+<robot name="my_robot" xmlns:xacro="http://www.ros.org/wiki/xacro">
 <!--Every dimension is written once here-->
 <!--Chassis box-->
@@ -15,2 +16,58 @@
 <xacro:property name="caster_radius" value="0.05"/>
 <xacro:property name="caster_thickness" value="0.02"/>
+<!--Materials-->
+<material name="blue">
+  <color rgba="0.2 0.4 0.8 1.0"/>
+</material>
+<material name="dark_grey">
+  <color rgba="0.2 0.2 0.2 1.0"/>
+</material>
+<material name="light_grey">
+  <color rgba="0.7 0.7 0.7 1.0"/>
+</material>
+<!--Wheel macro that have both the link and the joint,and takes a names and
+position-->
+<xacro:macro name="drive_wheel" params="prefix x_offset y_offset">
+<!--The cylinder stays upright. The joint below lays it flat -->
+  <link name="${prefix}_wheel">
+    <visual>
+      <origin xyz="0 0 0" rpy="0 0 0"/>
+      <geometry>
+        <cylinder radius="${wheel_radius}" length="${wheel_thickness}"/>
+      </geometry>
+      <material name="dark_grey"/>
+    </visual>
+  </link>
+   <!--The rpy lays the cylinder flat and points its z sideways, making z
+  the rolling axis.-->
+  <joint name=${prefix}_wheel_joint" type="continuous">
+    <parent link="base_link"/>
+    <child link="${prefix}_wheel"/>
+    <origin xyz=""${x_offset} ${y_offset} 0" rpy="${-pi/2} 0 0"/>
+    <axis xyz="0 0 1"/>
+  </joint>
+<!--============================ LINKS ============================-->
+<!--Root of the TF tree-->
+<link name="base_footprint">
+<!--Body of the robot-->
+<link name="base_link">
+  <visual>
+    <origin xyz="0 0 0" rpy="0 0 0"/>
+    <geometry>
+      <box size="${base_length} ${base_width} ${base_height}"/>
+    </geometry>
+    <material name="blue"/>
+  </visual>
+</link>
+<!--Front caster-->
+<link name="caster_wheel">
+  <visual>
+    <origin xyz="0 0 0" rpy="0 0 0"/>
+    <geometry>
+      <sphere radius="${caster_radius}"/>
+    </geometry>
+    <material name="light_grey"/>
+  </visual>
+</link>
+<!--============================ JOINTS ===========================-->
+<!--============================ WHEELS ===========================-->

Commit message: Add joints for base and caster, and update wheel definitions in my_robot.xacro

File: ros2_ws/src/assignment2/urdf/my_robot .urdf.xacro (robot description, xacro)
@@ -71,3 +71,23 @@
 </link>
 <!--============================ JOINTS ===========================-->
+<!--One wheel radius up, which is where the axle sits when the wheels
+touch the floor.-->
+<joint name="base_joint" type="fixed">
+  <parent link="base_footprint"/>
+  <child link="base_link"/>
+  <origin xyz="0 0 ${wheel_radius}" rpy="0 0 0"/>
+</joint>
+<!--Drops the caster until its underside reaches the ground.-->
+<joint name="caster_joint" type="fixed">
+  <parent link="base_link"/>
+  <child link="caster_wheel"/>
+  <origin xyz="${caster_x_offset} 0 ${caster_radius - wheel_radius}" rpy="0 0 0"/>
+</joint>
 <!--============================ WHEELS ===========================-->
+<!--Each call expands to a wheel link and its joint. Same axle, mirrored
+either side of the centre line.-->
+<xacro:drive_wheel prefix="left" x_offset="${wheel_x_offset}"
+                   y_offset="${wheel_separation/2}"/>
+<xacro:drive_wheel prefix="right" x_offset="${wheel_x_offset}"
+                   y_offset="${-wheel_separation/2}"/>
+</robot>
