Commit message: Add collision and inertial properties for robot components; include gazebo_control.xacro for simulation settings

File: ros2_ws/src/assignment2/urdf/gazebo_control.xacro (robot description, xacro)
@@ -7,5 +7,4 @@
         <mu2>0.0</mu2>
     </gazebo>
-<xacro:include filename="parameters.xacro"/
     <gazebo>
         <!--Turns cmd_vel into wheel rotation. Separation and radius

File: ros2_ws/src/assignment2/urdf/my_robot.urdf.xacro (robot description, xacro)
@@ -8,4 +8,6 @@
   <!--The robot: wheel macro, links and joints.-->
   <xacro:include filename="my_robot_core.xacro"/>
+  <!--Gazebo specific settings: friction and the simulation plugins.-->
+  <xacro:include filename="gazebo_control.xacro"/>
   <!--Task 2 adds gazebo_control.xacro here, Task 3 adds lidar.xacro.-->
 </robot>

File: ros2_ws/src/assignment2/urdf/my_robot_core.xacro (robot description, xacro)
@@ -15,4 +15,12 @@
       <material name="dark_grey"/>
     </visual>
+    <collision>
+      <origin xyz="0 0 0" rpy="0 0 0"/>
+      <geometry>
+        <cylinder radius="${wheel_radius}" length="${wheel_thickness}"/>
+      </geometry>
+    </collision>
+    <xacro:inertial_cylinder mass="${wheel_mass}" radius="${wheel_radius}"
+                             length="${wheel_thickness}"/>
   </link>
    <!--The rpy lays the cylinder flat and points its z sideways, making z
@@ -37,4 +45,12 @@
     <material name="blue"/>
   </visual>
+  <collision>
+    <origin xyz="0 0 0" rpy="0 0 0"/>
+    <geometry>
+      <box size="${base_length} ${base_width} ${base_height}"/>
+    </geometry>
+  </collision>
+  <xacro:inertial_box mass="${base_mass}" length="${base_length}"
+                      width="${base_width}" height="${base_height}"/>
 </link>
 <!--Front caster-->
@@ -47,4 +63,11 @@
     <material name="light_grey"/>
   </visual>
+  <collision>
+    <origin xyz="0 0 0" rpy="0 0 0"/>
+    <geometry>
+      <sphere radius="${caster_radius}"/>
+    </geometry>
+  </collision>
+  <xacro:inertial_sphere mass="${caster_mass}" radius="${caster_radius}"/>
 </link>
 <!--============================ JOINTS ===========================-->

File: ros2_ws/src/assignment2/urdf/parameters.xacro (robot description, xacro)
@@ -28,3 +28,33 @@
   <color rgba="0.7 0.7 0.7 1.0"/>
 </material>
+<!--Masses-->
+<xacro:property name="base_mass" value="5.0"/>
+<xacro:property name="wheel_mass" value="0.5"/>
+<xacro:property name="caster_mass" value="0.2"/>
+<!--Tensor for the primitive shapes.
+Each takes a mass and the dimensions.-->
+<xacro:macro name="inertial_box" params="mass length width height">
+  <inertial>
+    <mass value="${mass}"/>
+    <inertia ixx="${mass*(width*width + height*height)/12}" ixy="0" ixz="0"
+             iyy="${mass*(length*length + height*height)/12}" iyz="0"
+             izz="${mass*(length*length + width*width)/12}"/>
+  </inertial>
+</xacro:macro>
+<xacro:macro name="inertial_cylinder" params="mass radius length">
+  <inertial>
+    <mass value="${mass}"/>
+    <inertia ixx="${mass*(3*radius*radius + length*length)/12}" ixy="0" ixz="0"
+             iyy="${mass*(3*radius*radius + length*length)/12}" iyz="0"
+             izz="${mass*radius*radius/2}"/>
+  </inertial>
+</xacro:macro>
+<xacro:macro name="inertial_sphere" params="mass radius">
+  <inertial>
+    <mass value="${mass}"/>
+    <inertia ixx="${2*mass*radius*radius/5}" ixy="0" ixz="0"
+             iyy="${2*mass*radius*radius/5}" iyz="0"
+             izz="${2*mass*radius*radius/5}"/>
+  </inertial>
+</xacro:macro>
 </robot>
