Commit message: Update URDF and setup files for assignment3: add mesh support and fix link references

File: ros2_ws/src/assignment3/urdf/gazebo_control.xacro (robot description, xacro)
@@ -3,5 +3,5 @@
 <robot xmlns:xacro="http://www.ros.org/wiki/xacro">
     <!--Friction for caster wheel set to near zero-->
-    <gazebo reference="caster_wheel">
+    <gazebo reference="caster_wheel_link">
         <mu1>0.0</mu1>
         <mu2>0.0</mu2>

File: ros2_ws/src/assignment3/urdf/my_robot_core.xacro (robot description, xacro)
@@ -7,5 +7,5 @@
 <xacro:macro name="drive_wheel" params="prefix x_offset y_offset">
 <!--The cylinder stays upright. The joint below lays it flat -->
-  <link name="${prefix}_wheel">
+  <link name="${prefix}_wheel_link">
     <visual>
       <origin xyz="0 0 0" rpy="0 0 0"/>
@@ -28,5 +28,5 @@
   <joint name="${prefix}_wheel_joint" type="continuous">
     <parent link="base_link"/>
-    <child link="${prefix}_wheel"/>
+    <child link="${prefix}_wheel_link"/>
     <origin xyz="${x_offset} ${y_offset} 0" rpy="${-pi/2} 0 0"/>
     <axis xyz="0 0 1"/>
@@ -55,5 +55,5 @@
 </link>
 <!--Front caster-->
-<link name="caster_wheel">
+<link name="caster_wheel_link">
   <visual>
     <origin xyz="0 0 0" rpy="0 0 0"/>
@@ -80,7 +80,7 @@
 </joint>
 <!--Drops the caster until its underside reaches the ground.-->
-<joint name="caster_joint" type="fixed">
+<joint name="caster_wheel_joint" type="fixed">
   <parent link="base_link"/>
-  <child link="caster_wheel"/>
+  <child link="caster_wheel_link"/>
   <origin xyz="${caster_x_offset} 0 ${caster_radius - wheel_radius}" rpy="0 0 0"/>
 </joint>
