Commit message: Add origin elements to inertial macros for cylinder and sphere

File: ros2_ws/src/assignment3/urdf/parameters.xacro (robot description, xacro)
@@ -43,4 +43,5 @@
 <xacro:macro name="inertial_cylinder" params="mass radius length">
   <inertial>
+    <origin xyz="0 0 0" rpy="0 0 0"/>
     <mass value="${mass}"/>
     <inertia ixx="${mass*(3*radius*radius + length*length)/12}" ixy="0" ixz="0"
@@ -51,4 +52,5 @@
 <xacro:macro name="inertial_sphere" params="mass radius">
   <inertial>
+    <origin xyz="0 0 0" rpy="0 0 0"/>
     <mass value="${mass}"/>
     <inertia ixx="${2*mass*radius*radius/5}" ixy="0" ixz="0"
