Commit message: Update URDF files to replace cylinder geometries with mesh models for lidar, wheels, and body

File: ros2_ws/src/assignment3/urdf/lidar.xacro (robot description, xacro)
@@ -7,7 +7,6 @@
             <origin xyz="0 0 0" rpy="0 0 0"/>
             <geometry>
-                <cylinder radius="${lidar_radius}" length="${lidar_length}"/>
+                <mesh filename="${mesh_dir}/doomba_lidar.dae"/>
             </geometry>
-            <material name="dark_grey"/>
         </visual>
         <collision>

File: ros2_ws/src/assignment3/urdf/my_robot_core.xacro (robot description, xacro)
@@ -11,7 +11,6 @@
       <origin xyz="0 0 0" rpy="0 0 0"/>
       <geometry>
-        <cylinder radius="${wheel_radius}" length="${wheel_thickness}"/>
+        <mesh filename="${mesh_dir}/doomba_wheel.dae"/>
       </geometry>
-      <material name="dark_grey"/>
     </visual>
     <collision>
@@ -41,7 +40,6 @@
     <origin xyz="0 0 0" rpy="0 0 0"/>
     <geometry>
-      <box size="${base_length} ${base_width} ${base_height}"/>
+      <mesh filename="${mesh_dir}/doomba_body.dae"/>
     </geometry>
-    <material name="blue"/>
   </visual>
   <collision>

File: ros2_ws/src/assignment3/urdf/parameters.xacro (robot description, xacro)
@@ -3,4 +3,7 @@
 refers to these values.-->
 <robot xmlns:xacro="http://www.ros.org/wiki/xacro">
+<!--Shortcut to the mesh folder, so each visual only writes a file name.
+$(find assignment3) is the installed package path, filled in by xacro.-->
+<xacro:property name="mesh_dir" value="file://$(find assignment3)/meshes"/>
 <!--Every dimension is written once here-->
 <!--Chassis box-->

Commit message: Refactor LiDAR and robot core URDF files: update dimensions, improve comments, and fix geometry references

File: ros2_ws/src/assignment3/urdf/lidar.xacro (robot description, xacro)
@@ -13,15 +13,17 @@
             <origin xyz="0 0 0" rpy="0 0 0"/>
             <geometry>
-                <cylinder radius="${lidar_radius}" length="${lidar_length}"/>
+                <cylinder radius="${lidar_radius}" length="${lidar_height}"/>
             </geometry>
         </collision>
         <xacro:inertial_cylinder mass="${lidar_mass}" radius="${lidar_radius}"
-                                 length="${lidar_length}"/>
+                                 length="${lidar_height}"/>
     </link>
-    <!--Sits on the chasis roof: half the body up, then half the sensor-->
+    <!--Sits on the chassis roof, ahead of centre: half the body up, then
+    half the sensor-->
     <joint name="lidar_joint" type="fixed">
         <parent link="base_link"/>
         <child link="lidar_link"/>
-        <origin xyz="0 0 ${base_height/2 + lidar_length/2}" rpy="0 0 0"/>
+        <origin xyz="${lidar_x_offset} 0 ${base_height/2 + lidar_height/2}"
+                rpy="0 0 0"/>
     </joint>
     <gazebo reference="lidar_link">

File: ros2_ws/src/assignment3/urdf/my_robot_core.xacro (robot description, xacro)
@@ -1,10 +1,11 @@
 <?xml version="1.0"?>
 <!--The robot itself: the wheel macro, then the links and joints. Uses the
-dimensions and materials from parameters.urdf.xacro.-->
+dimensions and materials from parameters.xacro.-->
 <robot xmlns:xacro="http://www.ros.org/wiki/xacro">
-<!--Wheel macro that have both the link and the joint,and takes a names and
-position-->
+<!--Wheel macro that holds both the link and the joint, and takes a name and
+a position-->
 <xacro:macro name="drive_wheel" params="prefix x_offset y_offset">
-<!--The cylinder stays upright. The joint below lays it flat -->
+<!--The mesh and the collision cylinder both stand upright here. The joint
+below lays them flat.-->
   <link name="${prefix}_wheel_link">
     <visual>
@@ -23,10 +24,11 @@
                              length="${wheel_thickness}"/>
   </link>
-   <!--The rpy lays the cylinder flat and points its z sideways, making z
-  the rolling axis.-->
+  <!--The rpy lays the cylinder flat and points its z sideways, making z
+  the rolling axis. The height drops the wheel until it rests on the floor.-->
   <joint name="${prefix}_wheel_joint" type="continuous">
     <parent link="base_link"/>
     <child link="${prefix}_wheel_link"/>
-    <origin xyz="${x_offset} ${y_offset} 0" rpy="${-pi/2} 0 0"/>
+    <origin xyz="${x_offset} ${y_offset} ${wheel_radius - base_z}"
+            rpy="${-pi/2} 0 0"/>
     <axis xyz="0 0 1"/>
   </joint>
@@ -35,5 +37,7 @@
 <!--Root of the TF tree-->
 <link name="base_footprint"/>
-<!--Body of the robot-->
+<!--Body of the robot. Drawn with the mesh, but its physics come from the
+collision cylinder, which is kept at exactly the height on the diagram so
+the scan plane clears the roof.-->
 <link name="base_link">
   <visual>
@@ -46,11 +50,12 @@
     <origin xyz="0 0 0" rpy="0 0 0"/>
     <geometry>
-      <box size="${base_length} ${base_width} ${base_height}"/>
+      <cylinder radius="${base_radius}" length="${base_height}"/>
     </geometry>
   </collision>
-  <xacro:inertial_box mass="${base_mass}" length="${base_length}"
-                      width="${base_width}" height="${base_height}"/>
+  <xacro:inertial_cylinder mass="${base_mass}" radius="${base_radius}"
+                           length="${base_height}"/>
 </link>
-<!--Front caster-->
+<!--Front caster. The only link with no mesh, so it keeps the sphere for
+both the visual and the collision.-->
 <link name="caster_wheel_link">
   <visual>
@@ -70,10 +75,10 @@
 </link>
 <!--============================ JOINTS ===========================-->
-<!--Lifts the body off the ground. The lift is one wheel radius, so the
-wheels end up resting exactly on the floor.-->
+<!--Lifts the body off the ground: the clearance, plus half the body, puts
+the chassis centre at its ride height.-->
 <joint name="base_joint" type="fixed">
   <parent link="base_footprint"/>
   <child link="base_link"/>
-  <origin xyz="0 0 ${wheel_radius}" rpy="0 0 0"/>
+  <origin xyz="0 0 ${base_z}" rpy="0 0 0"/>
 </joint>
 <!--Drops the caster until its underside reaches the ground.-->
@@ -81,8 +86,9 @@
   <parent link="base_link"/>
   <child link="caster_wheel_link"/>
-  <origin xyz="${caster_x_offset} 0 ${caster_radius - wheel_radius}" rpy="0 0 0"/>
+  <origin xyz="${caster_x_offset} 0 ${caster_radius - base_z}" rpy="0 0 0"/>
 </joint>
 <!--============================ WHEELS ===========================-->
-<!--The two drive wheels, both built from the macros-->
+<!--The two drive wheels, both built from the macro. Half the track width
+each side of the centre line.-->
 <xacro:drive_wheel prefix="left" x_offset="${wheel_x_offset}"
                    y_offset="${wheel_separation/2}"/>

File: ros2_ws/src/assignment3/urdf/parameters.xacro (robot description, xacro)
@@ -1,52 +1,44 @@
 <?xml version="1.0"?>
-<!--Dimensions and materials. Included first, because everything below it
-refers to these values.-->
+<!--Dimensions, masses and materials. Included first, because everything below
+it refers to these values.-->
 <robot xmlns:xacro="http://www.ros.org/wiki/xacro">
 <!--Shortcut to the mesh folder, so each visual only writes a file name.
 $(find assignment3) is the installed package path, filled in by xacro.-->
 <xacro:property name="mesh_dir" value="file://$(find assignment3)/meshes"/>
-<!--Every dimension is written once here-->
-<!--Chassis box-->
-<xacro:property name="base_length" value="0.6"/>
-<xacro:property name="base_width" value="0.4"/>
-<xacro:property name="base_height" value="0.1"/>
-<!--Drive wheels-->
-<xacro:property name="wheel_radius" value="0.1"/>
-<xacro:property name="wheel_thickness" value="0.1"/>
-<!--How far behind the chassis centre the wheel sit-->
-<xacro:property name="wheel_x_offset" value="-0.1"/>
-<!--Distance between the two wheel centres-->
-<xacro:property name="wheel_separation" value="${base_width + wheel_thickness}"/>
-<!--Front caster-->
-<xacro:property name="caster_radius" value="0.05"/>
-<xacro:property name="caster_x_offset" value="0.2"/>
-<!--Materials-->
-<material name="blue">
-  <color rgba="0.2 0.4 0.8 1.0"/>
-</material>
-<material name="dark_grey">
-  <color rgba="0.2 0.2 0.2 1.0"/>
-</material>
+<!--============ SIZES, READ OFF THE DIAGRAM ============-->
+<!--Numbers from assigment3-->
+<!--Chassis: 32 cm across and 6 cm tall, riding 2 cm off the ground-->
+<xacro:property name="base_radius" value="0.16"/>
+<xacro:property name="base_height" value="0.06"/>
+<xacro:property name="ground_clearance" value="0.02"/>
+<!--Drive wheels: 6 cm across, 2.5 cm wide, 26 cm apart, 3 cm behind centre-->
+<xacro:property name="wheel_radius" value="0.03"/>
+<xacro:property name="wheel_thickness" value="0.025"/>
+<xacro:property name="wheel_separation" value="0.26"/>
+<xacro:property name="wheel_x_offset" value="-0.03"/>
+<!--Caster: 4 cm sphere, 12 cm ahead of centre-->
+<xacro:property name="caster_radius" value="0.02"/>
+<xacro:property name="caster_x_offset" value="0.12"/>
+<!--LiDAR: 6 cm across, 1 cm tall, 8 cm ahead of centre-->
+<xacro:property name="lidar_radius" value="0.03"/>
+<xacro:property name="lidar_height" value="0.01"/>
+<xacro:property name="lidar_x_offset" value="0.08"/>
+<!--============ WORKED OUT FROM THE SIZES ============-->
+<!--Height of the chassis centre above the ground. Every part below hangs
+off this one value, so raising the robot moves the whole body together.-->
+<xacro:property name="base_z" value="${ground_clearance + base_height/2}"/>
+<!--============ MASSES, FROM THE LINK TABLE ============-->
+<xacro:property name="base_mass" value="5.0"/>
+<xacro:property name="wheel_mass" value="0.2"/>
+<xacro:property name="caster_mass" value="0.1"/>
+<xacro:property name="lidar_mass" value="0.1"/>
+<!--============ MATERIALS ============-->
+<!--Only the caster needs one. The other links are drawn with meshes,
+which carry their own colours.-->
 <material name="light_grey">
   <color rgba="0.7 0.7 0.7 1.0"/>
 </material>
-<!--Masses-->
-<xacro:property name="base_mass" value="5.0"/>
-<xacro:property name="wheel_mass" value="0.5"/>
-<xacro:property name="caster_mass" value="0.2"/>
-<!--LiDAR-->
-<xacro:property name="lidar_mass" value="0.1"/>
-<xacro:property name="lidar_radius" value="0.05"/>
-<xacro:property name="lidar_length" value="0.1"/>
-<!--Tensor for the primitive shapes.
-Each takes a mass and the dimensions.-->
-<xacro:macro name="inertial_box" params="mass length width height">
-  <inertial>
-    <mass value="${mass}"/>
-    <inertia ixx="${mass*(width*width + height*height)/12}" ixy="0" ixz="0"
-             iyy="${mass*(length*length + height*height)/12}" iyz="0"
-             izz="${mass*(length*length + width*width)/12}"/>
-  </inertial>
-</xacro:macro>
+<!--============ INERTIA ============-->
+<!--Tensor for the primitive shapes. Each takes a mass and the dimensions.-->
 <xacro:macro name="inertial_cylinder" params="mass radius length">
   <inertial>

Commit message: Add lidar parameters and maze runner node to launch configuration

File: ros2_ws/src/assignment3/urdf/lidar.xacro (robot description, xacro)
@@ -37,8 +37,8 @@
                 <scan>
                     <horizontal>
-                        <samples>640</samples>
+                        <samples>${lidar_rays}</samples>
                         <resolution>1</resolution>
-                        <min_angle>-1.396263</min_angle>
-                        <max_angle>1.396263</max_angle>
+                        <min_angle>${-lidar_half_fov}</min_angle>
+                        <max_angle>${lidar_half_fov}</max_angle>
                     </horizontal>
                     <vertical>

File: ros2_ws/src/assignment3/urdf/my_robot.urdf.xacro (robot description, xacro)
@@ -3,4 +3,8 @@
 content of its own, it only pulls the parts together in order.-->
 <robot name="my_robot" xmlns:xacro="http://www.ros.org/wiki/xacro">
+  <!--Scan shape of the LiDAR. Set from the launch file so the different
+  configurations can be swapped without editing the model.-->
+  <xacro:arg name="lidar_fov" default="180"/>
+  <xacro:arg name="lidar_rays" default="45"/>
   <!--Dimensions and materials. Must come first, since the parts below
   refer to these values.-->

File: ros2_ws/src/assignment3/urdf/parameters.xacro (robot description, xacro)
@@ -24,4 +24,8 @@
 <xacro:property name="lidar_height" value="0.01"/>
 <xacro:property name="lidar_x_offset" value="0.08"/>
+<!--Scan shape, taken from the arguments. Half the field of view is what the
+sensor needs, since it counts out from straight ahead in both directions.-->
+<xacro:property name="lidar_rays" value="${$(arg lidar_rays)}"/>
+<xacro:property name="lidar_half_fov" value="${radians($(arg lidar_fov)) / 2}"/>
 <!--============ WORKED OUT FROM THE SIZES ============-->
 <!--Height of the chassis centre above the ground. Every part below hangs
